Commit message: Rotating Camera

File: rosbot_ros/src/rosbot_description/urdf/rosbot.xacro (robot description, xacro)
@@ -16,5 +16,5 @@
     <pose>0 0 0.1 0 0 0</pose>
     <inertial>
-      <mass value="5"/>
+      <mass value="50"/>
       <origin xyz="0 0 0.04" rpy=" 0 0 0"/>
       <inertia ixx="0.01" ixy="0.01" ixz="0" iyy="0.01" iyz="0.01" izz="0.01" />
@@ -236,10 +236,21 @@
   </transmission>
   <!-- Orbbec Astra RGBD Camera -->
-  <joint name="astra_joint" type="fixed">
-    <axis xyz="0 0 0" />
+  <joint name="astra_joint" type="continuous">
+    <axis xyz="0 0 1"/>
+    <limit effort="1" velocity="10"/>
     <origin xyz="-0.03 0 0.18" rpy="0 0 0"/>
     <parent link="body_link"/>
     <child link="camera_link"/>
   </joint>
+  <transmission name="astra_trans" type="SimpleTransmission">
+    <type>transmission_interface/SimpleTransmission</type>
+    <actuator name="astra_motor">
+      <mechanicalInterface>1</mechanicalInterface>
+      <hardwareInterface>hardware_interface/EffortJointInterface</hardwareInterface>
+    </actuator>
+    <joint name="astra_joint">
+      <hardwareInterface>hardware_interface/EffortJointInterface</hardwareInterface>
+    </joint>
+  </transmission>
   <link name="camera_link">
     <collision>
